File: electronics/lighting-tile-pcb/Lighting Tile Circuit V3.kicad_pcb (KiCad board)
At the start: 4 copper layers, 90 x 77.9 mm, 75 parts, among them J1 Conn_01x02_Socket, J2 USB_C_Receptacle_USB2.0_14P, J3 Conn_01x05, J4 Conn_01x05, J5 Conn_01x05, J6 Conn_01x05, J7 Conn_01x05, J8 Conn_01x05, Q1 MMBT3904, SW1 SW_Push, U1 74HC4051, U2 ESP32-C3-MINI-1U, U3 BQ25170DSGR, U4 74HC4051, U5 74AHCT125, U6 AP2112K-3.3, U7 TPS2116DRL, U8 TPS61022, U9 MCP111T-270E/TT

Commit message: Add files via upload
Parts:
- added R23: 10kΩ, Resistor_SMD:R_0603_1608Metric_Pad0.98x0.95mm_HandSolder, F.Cu at (129.8, 106.2)
- added R24: 10kΩ, Resistor_SMD:R_0603_1608Metric_Pad0.98x0.95mm_HandSolder, F.Cu at (114.5, 95.6)
- moved H2 0.65 mm to (132.0, 64.0)
- moved H1 0.61 mm to (92.0, 64.0)
- moved H3 0.54 mm to (132.0, 134.0)
- moved H4 0.49 mm to (92.0, 134.0)
Connections:
- net /GPIO7 - A (U1) renamed /7-A (U1)
- net /GPIO8 - A (U4) renamed /8-A (U4)
Routing:
- net /3V3: track 124.0 -> 134.4 mm
- net /8-A (U4): track 20.8 -> 23.0 mm
- net /LED_DATA: track 21.2 -> 21.8 mm
- net GND: vias 30 -> 31
