File: electronics/lighting-tile-pcb/Lighting Tile Circuit V3.kicad_sch (KiCad schematic)
At the start: 75 parts, among them J1 Conn_01x02_Socket, J2 USB_C_Receptacle_USB2.0_14P, J3 Conn_01x05, J4 Conn_01x05, J5 Conn_01x05, J6 Conn_01x05, J7 Conn_01x05, J8 Conn_01x05, Q1 MMBT3904, SW1 SW_Push, U1 74HC4051, U2 ESP32-C3-MINI-1U, U3 BQ25170DSGR, U4 74HC4051, U5 74AHCT125, U6 AP2112K-3.3, U7 TPS2116DRL, U8 TPS61022, U9 MCP111T-270E/TT

Commit message: Add files via upload
Parts:
- added R23, R24: 10kΩ, Resistor_SMD:R_0603_1608Metric_Pad0.98x0.95mm_HandSolder, symbol Device:R
Connections:
- net 3V3: now also R23.1, R24.1
- net LED_DATA: now also R24.2
- net GPIO7 - A (U1) renamed 7-A (U1)
- net GPIO8 - A (U4) renamed 8-A (U4)
- net 8-A (U4): now also R23.2
Other:
- moved on the sheet: C3
